File: NoahFC/NoahFC.kicad_pcb (KiCad board)
At the start: 2 copper layers, 36 x 56 mm, 54 parts, among them J1 ALE, J10 GND, J11 SCK, J12 MISO, J13 VCC, J14 GND, J16 CAM, J17 VTX, J18 RESET, J2 ELE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

Commit message: update scheme / design and board
Parts:
- removed C1, C12, C13, C2: 22pF, Capacitor_SMD:C_0805_2012Metric
- removed J16: CAM, Connector_PinHeader_2.54mm:PinHeader_1x02_P2.54mm_Vertical
- added J3: CAM, Connector_PinHeader_2.54mm:PinHeader_1x03_P2.54mm_Vertical, F.Cu at (152.0, 106.1)
- C9: value 2200pF -> 2.2nF
- J17: footprint Connector_PinHeader_2.54mm:PinHeader_1x02_P2.54mm_Vertical -> Connector_PinHeader_2.54mm:PinHeader_1x03_P2.54mm_Vertical
- Y1: footprint Crystal:Crystal_SMD_3225-4Pin_3.2x2.5mm -> Crystal:Resonator_SMD_Murata_CSTxExxV-3Pin_3.0x1.1mm
- moved C10 34.5 mm to (119.8, 83.9), turned to 180 degrees
- moved U4 31.9 mm to (121.6, 89.5)
- moved C11 29.8 mm to (123.4, 83.9)
- moved D3 29.8 mm to (119.8, 95.2)
- moved R4 29.4 mm to (119.8, 97.2), turned to 0 degrees
- moved R6 27.8 mm to (123.3, 95.2)
- moved C7 25.7 mm to (139.6, 105.3), turned to 0 degrees
- moved R5 24.8 mm to (123.3, 97.2), turned to 180 degrees
- moved Y2 23.3 mm to (139.5, 101.2), turned to -90 degrees
- moved Y1 14.3 mm to (128.3, 92.0)
- moved R9 12.7 mm to (127.4, 108.4), turned to 180 degrees
- moved U5 12.0 mm to (131.7, 102.9), turned to -90 degrees
- moved C19 11.6 mm to (140.4, 108.3)
- moved J10 11.5 mm to (151.3, 112.1)
- moved J13 11.5 mm to (125.6, 112.1)
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Connections:
- J1 pad 1: ALERON -> GND_BEC
- J1 pad 3: GND_BEC -> ALERON
- J17 pad 2: Net-(J17-Pad2) -> unconnected-(J17-Pad2)
- J2 pad 1: ELEVATOR -> GND_BEC
- J2 pad 3: GND_BEC -> ELEVATOR
- J6 pad 1: THROTTLE -> GND_BEC
- J6 pad 3: GND_BEC -> THROTTLE
- J7 pad 1: PPM -> GND_BEC
- J7 pad 2: 5V -> 5V_BEC
- J7 pad 3: GND -> PPM
- R10 pad 2: Net-(J17-Pad2) -> Net-(R10-Pad2)
- Y1 pad 2: XTAL1 -> GND
- Y1 pad 3: (no net) -> XTAL1
- Y2 pad 2: XTAL2_OSD -> GND
- Y2 pad 3: (no net) -> XTAL2_OSD
Other:
- board size 36 x 56 mm -> 36 x 40 mm
- board text added: "NoahFC rev2"
- board text removed: "5V"
- board text removed: "DTR"
- board text removed: "GND"
- board text removed: "RX"
- board text removed: "SCL"
- board text removed: "SDA"
- board text removed: "TX"

Commit message: redesign board
Parts:
- removed C4: 1uF, Capacitor_SMD:C_0805_2012Metric
- removed C5: 10uF, Capacitor_SMD:C_0805_2012Metric
- removed J10, J14: GND, TestPoint:TestPoint_Pad_4.0x4.0mm
- removed J13: VCC, TestPoint:TestPoint_Pad_4.0x4.0mm
- removed U3: AMS1117-5.0, Package_TO_SOT_SMD:SOT-223-3_TabPin2
- J5: footprint TestPoint:TestPoint_Pad_4.0x4.0mm -> TestPoint:TestPoint_Pad_1.5x1.5mm
- moved R4 32.4 mm to (151.6, 91.1), turned to 180 degrees
- moved U4 28.3 mm to (149.6, 85.3)
- moved D3 27.9 mm to (147.4, 91.1)
- moved R6 22.0 mm to (141.0, 108.2), turned to -90 degrees
- moved C6 21.0 mm to (144.0, 85.7), turned to 90 degrees
- moved C7 19.6 mm to (139.0, 85.7), turned to -90 degrees
- moved R5 18.8 mm to (138.5, 108.2), turned to 90 degrees
- moved Y2 18.5 mm to (121.4, 97.6), turned to 180 degrees
- moved C11 18.2 mm to (141.5, 85.7), turned to 90 degrees
- moved C20 16.8 mm to (134.9, 85.8)
- moved J11 13.5 mm to (141.8, 102.0), turned to 90 degrees
- moved J12 13.5 mm to (139.6, 102.0)
- moved C21 13.4 mm to (130.8, 81.1)
- moved J5 12.2 mm to (134.8, 107.8)
- moved R10 11.8 mm to (132.3, 110.3), turned to 0 degrees
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Connections:
- net VCC renamed Net-(R5-Pad1)
- C21 pad 1: Net-(C21-Pad1) -> Net-(U6-Pad12)
- C21 pad 2: Net-(C21-Pad2) -> Net-(U6-Pad8)
- J1 pad 1: GND_BEC -> GND
- J1 pad 2: 5V_BEC -> 5V
- J2 pad 1: GND_BEC -> GND
- J2 pad 2: 5V_BEC -> 5V
- J6 pad 1: GND_BEC -> GND
- J6 pad 2: 5V_BEC -> 5V
- J7 pad 1: GND_BEC -> GND
- J7 pad 2: 5V_BEC -> 5V
- U1 pad 23: unconnected-(U1-Pad23) -> VOLTAGE_READ
- U1 pad 25: VOLTAGE_READ -> unconnected-(U1-Pad25)
- U6 pad 12: Net-(C21-Pad2) -> Net-(U6-Pad12)
- U6 pad 8: Net-(C21-Pad1) -> Net-(U6-Pad8)
- Y2 pad 1: XTAL1_OSD -> XTAL2_OSD
- Y2 pad 3: XTAL2_OSD -> XTAL1_OSD
Routing:
- net GND: track 0.00 -> 223.1 mm, vias 0 -> 5
- net 5V: track 0.00 -> 121.4 mm, vias 0 -> 3
- net 3.3V: track 0.00 -> 66.4 mm, vias 0 -> 3
- net LED_GPS: track 0.00 -> 57.7 mm, vias 0 -> 4
- net SS: track 0.00 -> 43.6 mm, vias 0 -> 2
- net SCK: track 0.00 -> 40.7 mm, vias 0 -> 2
- net MOSI: track 0.00 -> 38.1 mm, vias 0 -> 2
- net SDA: track 0.00 -> 36.7 mm, vias 0 -> 3
- net TX: track 0.00 -> 31.7 mm, vias 0 -> 1
- net SCL: track 0.00 -> 31.5 mm, vias 0 -> 3
- net MISO: track 0.00 -> 31.3 mm, vias 0 -> 2
- net GPS_TX: track 0.00 -> 31.3 mm, vias 0 -> 4
- net Net-(C17-Pad2): track 0.00 -> 26.9 mm
- net LED_MODE: track 0.00 -> 26.0 mm, vias 0 -> 2
- net RESET: track 0.00 -> 26.0 mm, vias 0 -> 4
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Other:
- board text added: "5V"
- board text added: "ALE"
- board text added: "BATT"
- board text added: "CAM"
- board text added: "DTR"
- board text added: "ELE"
- board text added: "FTDI"
- board text added: "GND"
- board text added: "GPS"
- board text added: "PPM"
- board text added: "RX"
- board text added: "THR"
- board text added: "TX"
- board text added: "VOUT"

Commit message: tidy board
Parts:
- moved J11 1.10 mm to (142.9, 102.1)
- moved J12 0.71 mm to (140.3, 102.1)
- moved D1 0.20 mm to (151.3, 79.8)
- moved R2 0.20 mm to (147.8, 79.8)
Routing:
- net MISO: track 31.3 -> 33.7 mm
- net SCK: track 40.7 -> 43.1 mm
- net LED_GPS: track 57.7 -> 58.4 mm
