File: NoahFC/NoahFC.kicad_sch (KiCad schematic)
At the start: 50 parts, among them J1 ALE, J10 GND, J11 SCK, J12 MISO, J13 VCC, J14 GND, J17 VTX, J18 RESET, J2 ELE, J3 CAM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

Commit message: redesign board
Parts:
- removed C4: 1uF, Capacitor_SMD:C_0805_2012Metric, symbol Device:C
- removed C5: 10uF, Capacitor_SMD:C_0805_2012Metric, symbol Device:C
- removed J10, J14: GND, TestPoint:TestPoint_Pad_4.0x4.0mm, symbol Connector:Conn_01x01_Female
- removed J13: VCC, TestPoint:TestPoint_Pad_4.0x4.0mm, symbol Connector:Conn_01x01_Female
- removed U3: AMS1117-5.0, Package_TO_SOT_SMD:SOT-223-3_TabPin2, symbol Regulator_Linear:AMS1117-5.0
- J5: footprint TestPoint:TestPoint_Pad_4.0x4.0mm -> TestPoint:TestPoint_Pad_1.5x1.5mm
Connections:
- net 5V_BEC is gone; now on net 5V: J1.2 (Pin_2), J2.2 (Pin_2), J6.2 (Pin_2), J7.2 (Pin_2)
- net GND_BEC is gone; now on net GND: J1.1 (Pin_1), J2.1 (Pin_1), J6.1 (Pin_1), J7.1 (Pin_1)
- net VOLTAGE_READ: now also U1.23 (PC0); no longer U1.25 (PC2)
- net XTAL1_OSD: now also Y2.3; no longer Y2.1
- net XTAL2_OSD: now also Y2.1; no longer Y2.3
- net at C21.1: now also U6.12 (SETC); no longer U6.8 (SETP)
- net at C21.2: now also U6.8 (SETP); no longer U6.12 (SETC)
- net VCC: no longer names the net of J5.1 (Pin_1), R5.1
- no-connect marks 23 -> 22
Other:
- moved on the sheet: U1, U2, U4, U5, U6

Commit message: tidy board
Connections:
- no-connect marks 22 -> 23
Changed lines of the file:
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@@
   (no_connect (at 228.6 116.84))
   (no_connect (at 254 142.24))
+  (no_connect (at 161.29 54.61))
   (no_connect (at 58.42 133.35))
   (no_connect (at 86.36 49.53))
@@
   )
   (symbol (lib_id "Connector:Conn_01x01_Female") (at 185.42 46.99 180) (unit 1)
-    (in_bom yes) (on_board yes) (fields_autoplaced)
+    (in_bom yes) (on_board yes)
     (property "Reference" "J5" (id 0) (at 184.15 48.2601 0)
       (effects (font (size 1.27 1.27)) (justify left) hide)
