File: hardware/NoahFC.kicad_sch (KiCad schematic)
At the start: 37 parts, among them J1 ALE, J13 OSD, J2 ELE, J3 COMM, J4 FTDI, J6 THR, J7 PPM, J8 GPS, U1 ATmega328, U2 MPU-6050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

Commit message: rev6 project
Parts:
- J3: footprint Connector_JST:JST_SH_BM04B-SRSS-TB_1x04-1MP_P1.00mm_Vertical -> Connector_JST:JST_SH_BM05B-SRSS-TB_1x05-1MP_P1.00mm_Vertical; symbol Connector:Conn_01x04_Socket -> Connector:Conn_01x05_Socket
Connections:
- net 5V: now also J3.2 (Pin_2); no longer J3.1 (Pin_1)
- net GND: now also J3.3 (Pin_3); no longer J3.2 (Pin_2)
- net SCL: now also J3.5 (Pin_5); no longer J3.4 (Pin_4)
- net SDA: now also J3.4 (Pin_4); no longer J3.3 (Pin_3)
- net THROTTLE: now also J3.1 (Pin_1)
