File: hardware/NoahFC.kicad_sch (KiCad schematic)
At the start: 46 parts, among them J1 ALE, J10 ESC-, J11 CAM, J12 VTX, J15 ESC_PWM, J17 BEC, J2 ELE, J3 VCC, J4 FTDI, J5 GND, J6 THR, J7 PPM, J8 GPS, J9 ESC+, U1 ATmega328, U3 XC6206, U4 LM317, U6 AT7456, Y1 16Mhz, Y3 27Mhz

Commit message: add rev10
Changed lines of the file:
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@@
 	(title_block
 		(title "NoahFC")
-		(rev "9")
+		(rev "10")
 	)
 	(text_box "JUMPERS\n"
@@
 	(wire
 		(pts
-			(xy 34.29 177.8) (xy 34.29 172.72)
-		)
-		(stroke
+			(xy 34.29 172.72) (xy 34.29 177.8)
+		)
+		(stroke
